File: NMX-201.sch (EAGLE design)
At the start: 61 parts, among them IC1 A4983TOP, IC2 A4983TOP, IC3 A4983TOP, J1 MOLEX-4-RA, J2 MOLEX-4-RA, J3 MOLEX-4-RA, U1 CADJ, U2 CADJ, U3 MOUNT-HOLE3.2, U4 MOUNT-HOLE3.2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

Commit message: Updated NMX-201 to match NMX-201B
The only difference between NMX-201 and NMX-201B is whether the the
component attached to the motor connector ports is a screw terminal or a
Molex connector, so there's really no need to maintain two different
schematics / board files. These differences should be reflected in the
BOM instead.
Parts:
- added S2, S3: CHS-02A, switch-copal:CHS-02A
- J1, J2, J3: value MOLEX-4-RA -> MOLEX-4-RAPRO-CONNECTOR; device QS_Components:MOLEX-4-RA -> NMX_StepperSide_V1-2:MOLEX-4-RAPRO-CONNECTOR
- R16, R17, R18: value 430 -> 14k; MPN RC0402FR-07430RL -> RC0402FR-0714KL
Connections:
- new net N$16: LED1.C, S2.4
- new net N$18: LED2.C, S2.3
- new net N$19: LED3.C, S3.4
- net AEN_1: now also S2.1; no longer LED1.C
- net AEN_2: now also S2.2; no longer LED2.C
- net AEN_3: now also S3.1; no longer LED3.C
Other:
- moved on the sheet: C15, C3, LED1, LED2, LED3, R16, R17, R18, R5
