File: NMX-201.sch (EAGLE design)
At the start: 63 parts, among them IC1 A4983TOP, IC2 A4983TOP, IC3 A4983TOP, J1 MOLEX-4-RAPRO-CONNECTOR, J2 MOLEX-4-RAPRO-CONNECTOR, J3 MOLEX-4-RAPRO-CONNECTOR, U1 CADJ, U2 CADJ, U3 MOUNT-HOLE3.2, U4 MOUNT-HOLE3.2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

Commit message: Changed several resistor values to reduce unique part count
See NMX-200 / NMX-201 BOM Google doc change log for 12/15/16 for
details.
Parts:
- R14, R5, R9: value 20k -> 10k
- R16, R17, R18: value 14k -> 10k
Changed lines of the file:
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@@
 <part name="GND35" library="SparkFun" deviceset="GND" device=""/>
 <part name="GND36" library="SparkFun" deviceset="GND" device=""/>
-<part name="R5" library="resistor" deviceset="R-US_" device="R0402_B" value="20k">
+<part name="R5" library="resistor" deviceset="R-US_" device="R0402_B" value="10k">
 <attribute name="MF" value="Yageo"/>
 <attribute name="MPN" value="RC0402FR-0720KL"/>
@@
 <part name="GND6" library="SparkFun" deviceset="GND" device=""/>
 <part name="GND7" library="SparkFun" deviceset="GND" device=""/>
-<part name="R9" library="resistor" deviceset="R-US_" device="R0402_B" value="20k">
+<part name="R9" library="resistor" deviceset="R-US_" device="R0402_B" value="10k">
 <attribute name="MF" value="Yageo"/>
 <attribute name="MPN" value="RC0402FR-0720KL"/>
@@
 <part name="GND15" library="SparkFun" deviceset="GND" device=""/>
 <part name="GND16" library="SparkFun" deviceset="GND" device=""/>
-<part name="R14" library="resistor" deviceset="R-US_" device="R0402_B" value="20k">
+<part name="R14" library="resistor" deviceset="R-US_" device="R0402_B" value="10k">
 <attribute name="MF" value="Yageo"/>
 <attribute name="MPN" value="RC0402FR-0720KL"/>
@@
 <attribute name="MPN" value="LB Q39G-L2N2-35-1"/>
 </part>
-<part name="R16" library="resistor" deviceset="R-US_" device="R0402_B" value="14k">
+<part name="R16" library="resistor" deviceset="R-US_" device="R0402_B" value="10k">
 <attribute name="MF" value="Yageo"/>
 <attribute name="MPN" value="RC0402FR-0714KL"/>
 </part>
-<part name="R17" library="resistor" deviceset="R-US_" device="R0402_B" value="14k">
+<part name="R17" library="resistor" deviceset="R-US_" device="R0402_B" value="10k">
 <attribute name="MF" value="Yageo"/>
 <attribute name="MPN" value="RC0402FR-0714KL"/>
 </part>
-<part name="R18" library="resistor" deviceset="R-US_" device="R0402_B" value="14k">
+<part name="R18" library="resistor" deviceset="R-US_" device="R0402_B" value="10k">
 <attribute name="MF" value="Yageo"/>
 <attribute name="MPN" value="RC0402FR-0714KL"/>
