File: NMX-201.brd (EAGLE design)
At the start: 50.8 x 50.2 mm, 63 parts, among them IC1 A4983TOP, IC2 A4983TOP, IC3 A4983TOP, J1 MOLEX-4-RAPRO-CONNECTOR, J2 MOLEX-4-RAPRO-CONNECTOR, J3 MOLEX-4-RAPRO-CONNECTOR, U1 CADJ, U2 CADJ, U3 MOUNT-HOLE3.2, U4 MOUNT-HOLE3.2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

Commit message: Changed several resistor values to reduce unique part count
See NMX-200 / NMX-201 BOM Google doc change log for 12/15/16 for
details.
Parts:
- R14, R5, R9: value 20k -> 10k
- R16, R17, R18: value 14k -> 10k
Changed lines of the file:
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@@
 <attribute name="VALUE" x="12.47775" y="39.33825" size="0.8128" layer="27" rot="R180"/>
 </element>
-<element name="R5" library="resistor" package="R0402_BOTTOM" value="20k" x="14.605" y="26.67" smashed="yes" rot="MR0">
+<element name="R5" library="resistor" package="R0402_BOTTOM" value="10k" x="14.605" y="26.67" smashed="yes" rot="MR0">
 <attribute name="MPN" value="RC0402FR-0720KL" x="-14.605" y="-34.29" size="1.778" layer="28" rot="MR0" display="off"/>
 <attribute name="MF" value="Yageo" x="-14.605" y="-34.29" size="1.778" layer="28" rot="MR0" display="off"/>
@@
 <attribute name="VALUE" x="21.209" y="23.78075" size="0.8128" layer="27" rot="R180"/>
 </element>
-<element name="R9" library="resistor" package="R0402_BOTTOM" value="20k" x="30.48" y="15.875" smashed="yes" rot="R270">
+<element name="R9" library="resistor" package="R0402_BOTTOM" value="10k" x="30.48" y="15.875" smashed="yes" rot="R270">
 <attribute name="MPN" value="RC0402FR-0720KL" x="-30.48" y="-20.955" size="1.778" layer="27" rot="R270" display="off"/>
 <attribute name="MF" value="Yageo" x="-30.48" y="-20.955" size="1.778" layer="27" rot="R270" display="off"/>
@@
 <attribute name="VALUE" x="31.5595" y="38.7985" size="0.8128" layer="27" rot="R90"/>
 </element>
-<element name="R14" library="resistor" package="R0402_BOTTOM" value="20k" x="33.02" y="27.305" smashed="yes" rot="MR0">
+<element name="R14" library="resistor" package="R0402_BOTTOM" value="10k" x="33.02" y="27.305" smashed="yes" rot="MR0">
 <attribute name="MPN" value="RC0402FR-0720KL" x="-15.24" y="-33.655" size="1.778" layer="28" rot="MR0" display="off"/>
 <attribute name="MF" value="Yageo" x="-15.24" y="-33.655" size="1.778" layer="28" rot="MR0" display="off"/>
@@
 <attribute name="MPN" value="LB Q39G-L2N2-35-1" x="38.25875" y="48.26" size="1.778" layer="27" rot="R270" display="off"/>
 </element>
-<element name="R16" library="resistor" package="R0402_BOTTOM" value="14k" x="17.62125" y="48.41875" smashed="yes" rot="MR180">
+<element name="R16" library="resistor" package="R0402_BOTTOM" value="10k" x="17.62125" y="48.41875" smashed="yes" rot="MR180">
 <attribute name="MPN" value="RC0402FR-0714KL" x="17.62125" y="48.41875" size="1.778" layer="28" rot="MR180" display="off"/>
 <attribute name="MF" value="Yageo" x="17.62125" y="48.41875" size="1.778" layer="28" rot="MR180" display="off"/>
@@
 <attribute name="VALUE" x="18.25625" y="46.51375" size="0.8128" layer="27" rot="R180"/>
 </element>
-<element name="R17" library="resistor" package="R0402_BOTTOM" value="14k" x="20.955" y="48.41875" smashed="yes" rot="MR0">
+<element name="R17" library="resistor" package="R0402_BOTTOM" value="10k" x="20.955" y="48.41875" smashed="yes" rot="MR0">
 <attribute name="MPN" value="RC0402FR-0714KL" x="20.955" y="48.41875" size="1.778" layer="28" rot="MR0" display="off"/>
 <attribute name="MF" value="Yageo" x="20.955" y="48.41875" size="1.778" layer="28" rot="MR0" display="off"/>
@@
 <attribute name="VALUE" x="20.16125" y="45.75175" size="0.8128" layer="27"/>
 </element>
-<element name="R18" library="resistor" package="R0402_BOTTOM" value="14k" x="33.3375" y="48.41875" smashed="yes" rot="MR0">
+<element name="R18" library="resistor" package="R0402_BOTTOM" value="10k" x="33.3375" y="48.41875" smashed="yes" rot="MR0">
 <attribute name="MPN" value="RC0402FR-0714KL" x="33.3375" y="48.41875" size="1.778" layer="28" rot="MR0" display="off"/>
 <attribute name="MF" value="Yageo" x="33.3375" y="48.41875" size="1.778" layer="28" rot="MR0" display="off"/>
